Commit message: simulation up - with basic world and robot spawning

File: src/semantic_comm_runtime/assets/robot/semantic_robot.urdf (robot description, URDF)
Before this commit: robot semantic_robot, 4 links, 3 joints
Links:
- link left_wheel: geometry collision cylinder length=0.04 radius=0.15; visual cylinder length=0.04 radius=0.15
- link right_wheel: geometry collision cylinder length=0.04 radius=0.15; visual cylinder length=0.04 radius=0.15
